Commit message: 修正urdf关节限位Bug

File: galileo_mini_x5_description/urdf/galileo_mini_x5.urdf (robot description, URDF)
Before this commit: robot galileo_mini_description, 26 links, 25 joints
Joints:
- removed joint RR_foot_joint
- added joint HR_foot_joint: type fixed, parent HR_knee_link, child HR_foot_link, origin xyz=0.032939 0 -0.26149 rpy=0 0 0, axis 0 0 0
- joint FL_hip_joint: limit lower=-1.0472 upper=4.1888 effort=100 velocity=21 -> lower=-4.1888 upper=1.0472 effort=100 velocity=21
- joint FR_hip_joint: limit lower=-1.0472 upper=4.1888 effort=100 velocity=21 -> lower=-4.1888 upper=1.0472 effort=100 velocity=21
- joint HL_hip_joint: limit lower=-1.0472 upper=4.1888 effort=100 velocity=21 -> lower=-4.1888 upper=1.0472 effort=100 velocity=21
- joint HR_hip_joint: limit lower=-1.0472 upper=4.1888 effort=100 velocity=21 -> lower=-4.1888 upper=1.0472 effort=100 velocity=21

Commit message: 修正HL_foot_link为HL_foot_joint以确保关节名称一致性

File: galileo_mini_x5_description/urdf/galileo_mini_x5.urdf (robot description, URDF)
Before this commit: robot galileo_mini_description, 26 links, 25 joints
Joints:
- removed joint HL_foot_link
- added joint HL_foot_joint: type fixed, parent HL_knee_link, child HL_foot_link, origin xyz=0.0329385085367515 0 -0.261492891464613 rpy=0 0 0, axis 0 0 0
