Commit message: 修改x5机械臂的关节限位

File: galileo_v1d6_x5_description/urdf/galileo_v1d6_x5.urdf (robot description, URDF)
Before this commit: robot galileo_v1d6, 26 links, 25 joints
Joints:
- joint joint1: limit lower=-10 upper=10 effort=100 velocity=1000 -> lower=-3.14 upper=2.6 effort=100 velocity=1000
- joint joint2: limit lower=-10 upper=10 effort=100 velocity=1000 -> lower=-0.1 upper=3.6 effort=100 velocity=1000
- joint joint3: limit lower=-10 upper=10 effort=100 velocity=1000 -> lower=0 upper=3.14 effort=100 velocity=1000
- joint joint4: limit lower=-10 upper=10 effort=100 velocity=1000 -> lower=-1.3 upper=1.3 effort=100 velocity=1000
- joint joint5: limit lower=-10 upper=10 effort=100 velocity=1000 -> lower=-1.57 upper=1.57 effort=100 velocity=1000
- joint joint6: limit lower=-10 upper=10 effort=100 velocity=1000 -> lower=-2.1 upper=2.1 effort=100 velocity=1000

File: x5_description/urdf/x5.urdf (robot description, URDF)
Before this commit: robot x5_description, 9 links, 8 joints
Joints:
- joint joint1: limit lower=-10 upper=10 effort=100 velocity=1000 -> lower=-3.14 upper=2.6 effort=100 velocity=1000
- joint joint2: limit lower=-10 upper=10 effort=100 velocity=1000 -> lower=-0.1 upper=3.6 effort=100 velocity=1000
- joint joint3: limit lower=-10 upper=10 effort=100 velocity=1000 -> lower=0 upper=3.14 effort=100 velocity=1000
- joint joint4: limit lower=-10 upper=10 effort=100 velocity=1000 -> lower=-1.3 upper=1.3 effort=100 velocity=1000
- joint joint5: limit lower=-10 upper=10 effort=100 velocity=1000 -> lower=-1.57 upper=1.57 effort=100 velocity=1000
- joint joint6: limit lower=-10 upper=10 effort=100 velocity=1000 -> lower=-2.1 upper=2.1 effort=100 velocity=1000

Commit message: 更新galileo_v1d6_x5的简化碰撞模型

File: galileo_v1d6_x5_description/urdf/galileo_v1d6_x5.urdf (robot description, URDF)
Before this commit: robot galileo_v1d6, 26 links, 25 joints
Links:
- link link0: geometry collision cylinder length=0.06 radius=0.03; visual mesh filename=package://galileo_v1d6_x5_description/meshes/link0.STL
- link link1: geometry visual mesh filename=package://galileo_v1d6_x5_description/meshes/link1.STL
- link link2: geometry collision box size=0.22 0.06 0.05; collision cylinder length=0.06 radius=0.03
- link link3: geometry collision box size=0.19 0.05 0.04; collision cylinder length=0.05 radius=0.028
- link link4: geometry collision cylinder length=0.04 radius=0.03; visual mesh filename=package://galileo_v1d6_x5_description/meshes/link4.STL
- link link5: geometry collision cylinder length=0.04 radius=0.03; visual mesh filename=package://galileo_v1d6_x5_description/meshes/link5.STL
- link link6: geometry collision cylinder length=0.06 radius=0.03; visual mesh filename=package://galileo_v1d6_x5_description/meshes/link6.STL
