Commit message: 修正mesh文件

File: bqr3_arm_description/urdf/bqr3_arm.urdf (robot description, URDF)
Before this commit: robot bqr3_arm, 24 links, 23 joints
Links:
- link FL_abd_link: geometry collision mesh filename=package://bqr3_arm_description/meshes/FL_abd_link.STL; visual mesh filename=package://bqr3_arm_description/meshes/FL_abd_link.STL
- link FL_foot_link: geometry collision mesh filename=package://bqr3_arm_description/meshes/FL_foot_link.STL; visual mesh filename=package://bqr3_arm_description/meshes/FL_foot_link.STL
- link FL_hip_link: geometry collision mesh filename=package://bqr3_arm_description/meshes/FL_hip_link.STL; visual mesh filename=package://bqr3_arm_description/meshes/FL_hip_link.STL
- link FL_knee_link: geometry collision mesh filename=package://bqr3_arm_description/meshes/FL_knee_link.STL; visual mesh filename=package://bqr3_arm_description/meshes/FL_knee_link.STL
- link FR_abd_link: geometry collision mesh filename=package://bqr3_arm_description/meshes/FR_abd_link.STL; visual mesh filename=package://bqr3_arm_description/meshes/FR_abd_link.STL
- link FR_foot_link: geometry collision mesh filename=package://bqr3_arm_description/meshes/FR_foot_link.STL; visual mesh filename=package://bqr3_arm_description/meshes/FR_foot_link.STL
- link FR_hip_link: geometry collision mesh filename=package://bqr3_arm_description/meshes/FR_hip_link.STL; visual mesh filename=package://bqr3_arm_description/meshes/FR_hip_link.STL
- link FR_knee_link: geometry collision mesh filename=package://bqr3_arm_description/meshes/FR_knee_link.STL; visual mesh filename=package://bqr3_arm_description/meshes/FR_knee_link.STL
- link HL_abd_link: geometry collision mesh filename=package://bqr3_arm_description/meshes/HL_abd_link.STL; visual mesh filename=package://bqr3_arm_description/meshes/HL_abd_link.STL
- link HL_foot_link: geometry collision mesh filename=package://bqr3_arm_description/meshes/HL_foot_link.STL; visual mesh filename=package://bqr3_arm_description/meshes/HL_foot_link.STL
- link HL_hip_link: geometry collision mesh filename=package://bqr3_arm_description/meshes/HL_hip_link.STL; visual mesh filename=package://bqr3_arm_description/meshes/HL_hip_link.STL
- link HL_knee_link: geometry collision mesh filename=package://bqr3_arm_description/meshes/HL_knee_link.STL; visual mesh filename=package://bqr3_arm_description/meshes/HL_knee_link.STL
- link HR_abd_link: geometry collision mesh filename=package://bqr3_arm_description/meshes/HR_abd_link.STL; visual mesh filename=package://bqr3_arm_description/meshes/HR_abd_link.STL
- link HR_foot_link: geometry collision mesh filename=package://bqr3_arm_description/meshes/HR_foot_link.STL; visual mesh filename=package://bqr3_arm_description/meshes/HR_foot_link.STL
- link HR_hip_link: geometry collision mesh filename=package://bqr3_arm_description/meshes/HR_hip_link.STL; visual mesh filename=package://bqr3_arm_description/meshes/HR_hip_link.STL
- link HR_knee_link: geometry collision mesh filename=package://bqr3_arm_description/meshes/HR_knee_link.STL; visual mesh filename=package://bqr3_arm_description/meshes/HR_knee_link.STL
- link base_link: geometry collision mesh filename=package://bqr3_arm_description/meshes/base_link.STL; visual mesh filename=package://bqr3_arm_description/meshes/base_link.STL

Commit message: 更新部分简化碰撞模型

File: bqr3_arm_description/urdf/bqr3_arm.urdf (robot description, URDF)
Before this commit: robot bqr3_arm, 24 links, 23 joints
Links:
- link base_link: geometry collision box size=0.5 0.25 0.1; visual mesh filename=package://bqr3_arm_description/meshes/base_link.STL
- link forearm: geometry collision cylinder length=0.4 radius=0.02; visual mesh filename=package://bqr3_arm_description/meshes/forearm.STL
- link upper_arm: geometry collision cylinder length=0.38 radius=0.02; visual mesh filename=package://bqr3_arm_description/meshes/upper_arm.STL
- link wrist_pitch: geometry collision cylinder length=0.24 radius=0.02; visual mesh filename=package://bqr3_arm_description/meshes/wrist_pitch.STL
