Commit message: feat: 更新go2_sphere_collision.urdf，修改碰撞体几何形状为球体，调整原点位置，移除多余的碰撞体定义

File: go2_description/urdf/go2_sphere_collision.urdf (robot description, URDF)
Before this commit: robot go2_description, 29 links, 28 joints
Links:
- removed link FL_calflower
- removed link FL_calflower1
- removed link FR_calflower
- removed link FR_calflower1
- removed link RL_calflower
- removed link RL_calflower1
- removed link RR_calflower
- removed link RR_calflower1
- link FL_calf: geometry visual mesh filename=package://go2_description/dae/calf.dae
- link FL_hip: geometry collision sphere radius=0.05; visual mesh filename=package://go2_description/dae/hip.dae
- link FL_thigh: geometry collision sphere radius=0.025; visual mesh filename=package://go2_description/dae/thigh.dae
- link FR_calf: geometry visual mesh filename=package://go2_description/dae/calf_mirror.dae
- link FR_hip: geometry collision sphere radius=0.05; visual mesh filename=package://go2_description/dae/hip.dae
- link FR_thigh: geometry collision sphere radius=0.025; visual mesh filename=package://go2_description/dae/thigh_mirror.dae
- link RL_calf: geometry visual mesh filename=package://go2_description/dae/calf.dae
- link RL_hip: geometry collision sphere radius=0.05; visual mesh filename=package://go2_description/dae/hip.dae
- link RL_thigh: geometry collision sphere radius=0.025; visual mesh filename=package://go2_description/dae/thigh.dae
- link RR_calf: geometry visual mesh filename=package://go2_description/dae/calf_mirror.dae
- link RR_hip: geometry collision sphere radius=0.05; visual mesh filename=package://go2_description/dae/hip.dae
- link RR_thigh: geometry collision sphere radius=0.025; visual mesh filename=package://go2_description/dae/thigh_mirror.dae
Joints:
- removed joint FL_calflower1_joint
- removed joint FL_calflower_joint
- removed joint FR_calflower1_joint
- removed joint FR_calflower_joint
- removed joint RL_calflower1_joint
- removed joint RL_calflower_joint
- removed joint RR_calflower1_joint
- removed joint RR_calflower_joint
