Commit message: 自定义x5机械臂的简化碰撞模型

File: x5_description/urdf/x5.urdf (robot description, URDF)
Before this commit: robot x5_description, 9 links, 8 joints
Links:
- link link0: geometry collision cylinder length=0.06 radius=0.03; visual mesh filename=package://x5_description/meshes/link0.STL
- link link1: geometry visual mesh filename=package://x5_description/meshes/link1.STL
- link link2: geometry collision box size=0.22 0.06 0.05; collision cylinder length=0.06 radius=0.03
- link link3: geometry collision box size=0.19 0.05 0.04; collision cylinder length=0.05 radius=0.028
- link link4: geometry collision cylinder length=0.04 radius=0.03; visual mesh filename=package://x5_description/meshes/link4.STL
- link link5: geometry collision cylinder length=0.04 radius=0.03; visual mesh filename=package://x5_description/meshes/link5.STL
- link link6: geometry collision cylinder length=0.06 radius=0.03; visual mesh filename=package://x5_description/meshes/link6.STL

Commit message: 增加一些模型

File: x5_description/urdf/x5.urdf (robot description, URDF)
Before this commit: robot x5_description, 9 links, 8 joints
Links:
- link link7: geometry collision box size=0.03 0.004 0.036; collision box size=0.04 0.004 0.0105
- link link8: geometry collision box size=0.03 0.004 0.036; collision box size=0.04 0.004 0.0105
